File: DogTracker.kicad_sch (KiCad schematic)
At the start: 7 parts

Commit message: update symbols
Parts:
- added C?: C_Small, symbol Device:C_Small
- added C?: 1uF, symbol Device:C_Small
- added R?: 220, symbol Device:R_US
- added R? (x3): 10k, symbol Device:R_US
- added R? (x2): 2.2k, symbol Device:R_US
- added U?: Origin_GPS1410, symbol DogTracker:Origin_GPS1410
- added U?: ADP160AUJZ-1.8-R7, symbol DogTracker:ADP160AUJZ-2.8-R7
- added U?: SN74AUP1T97, symbol DogTracker:SN74AUP1T97
- added U?: NFA18SL407V1A45L, symbol DogTracker:NFA18SL407V1A45L
Connections:
- net GND: now also C?.2, C?.2, R?.2, R?.2, U?.1 (GND), U?.2 (GND), U?.2 (GND), U?.2 (GND), U?.5 (GND)
- new net: R?.1, R?.2, U?.1 (ON/OFF)
- new net: R?.1, U?. (9), U?.10 (RX)
- new net: R?.1, U?. (9), U?.3 (TX)
- new net: R?.1, U?. (9), U?.7 (CTS)
- new net: R?.1, U?. (9), U?.9 (RTS)
- new net: C?.1, U?.5 (Vout)
- new net: C?.1, U?.1 (Vin)
- new net 1.8V: R?.2, R?.2
- new net 1PPS_GPS: U?.2 (1PPS)
- new net GPS_ON: R?.1
- new net I2C_SCL: U?. (9), U?.1 (IN_B), U?.3 (IN_A), U?.6 (IN_C)
- new net I2C_SDA: U?. (9)
- new net RESET: U?.8 (RESET)
- new net SPI_CLK: U?. (9)
- new net SPI_nCS: U?. (9)
- new net VCC: U?.4 (VCC), U?.5 (VCC)
- new net Vi/o: R?.2
- new net WAKEUP_GPS: U?.6 (WAKEUP)

Commit message: 'updated feather'
Parts:
- removed U?: ItsyBitsy, symbol DogTracker:ItsyBitsy
- added BT?: Battery, symbol Device:Battery
- added IC?: M4 Feather, 3857, symbol DogTracker:M4 Feather
Connections:
- net 1.8V is gone; now on net +1V8: R?.2, R?.2
- net SPI_CLK is gone; now on net I2C_SDA: U?. (9)
- net SPI_nCS is gone; now on net I2C_SDA: U?. (9)
- net Vi/o is gone; now on net +1V8: R?.2
- net GND: now also IC?.13 (GND)
- net I2C_SDA: now also IC?.28 (SDA)
- net LORA_CS: now also IC?.1 (D4)
- net MISO: now also IC?.5 (MOSI)
- net MOSI: now also IC?.4 (MISO)
- net PED_CS: now also IC?.20 (D13)
- net SCK: now also IC?.6 (SCK)
- net Speaker: now also IC?.21 (D12)
- net +1V8: now reaches C?.1, U?.5 (Vout)
- net VDD: now reaches C?.1, U?.1 (Vin)
- net VDD: now also IC?.15 (+3V3)
- no-connect marks 9 -> 7
Other:
- moved on the sheet: C?, U?

Commit message: add text, hope this works
Other:
- note added: "GPS"
- note added: "LORA"
- note added: "MCU"
Changed lines of the file:
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@@
     (stroke (width 0) (type default) (color 0 0 0 0))
+  )
+  (text "GPS" (at 63.5 134.62 0)
+    (effects (font (size 1.27 1.27)) (justify left bottom))
+  )
+  (text "LORA" (at 81.28 20.32 0)
+    (effects (font (size 1.27 1.27)) (justify left bottom))
+  )
+  (text "MCU" (at 228.6 91.44 0)
+    (effects (font (size 1.27 1.27)) (justify left bottom))
   )
   (label "I2C_SCL" (at 157.48 161.29 0)

Commit message: 'rearrange schematic'
Connections:
- net at R?.1, U?. (9), U?.10 (RX): now also R?.1, U?.7 (CTS)
Other:
- moved on the sheet: BT?, C?, IC?, LS?, R?, U?
