File: Hardware/Kicad/Dog_Tracker.kicad_pcb (KiCad board)
At the start: 4 copper layers, 100 x 53.9 mm, 22 parts, among them IC1 M4 Feather, U1 ADP160AUJZ-1.8-R7, U2 SX1280IMLTRT, U3 Origin_GPS1510, U5 SN74AUP1T97, U6 LSM6DSO32

Commit message: 'sent for fab'
Routing:
- net GND: track 36.6 -> 54.6 mm, vias 63 -> 65
Changed lines of the file:
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@@
     (property "Sheetname" "")
     (attr through_hole)
-    (fp_text reference "LS1" (at 0.381 13.843 180 unlocked) (layer "B.SilkS")
+    (fp_text reference "LS1" (at 0.381 15.9 180 unlocked) (layer "B.SilkS")
       (effects (font (size 1 1) (thickness 0.15)) (justify mirror))
     )
@@
       (effects (font (size 1 1) (thickness 0.15)) (justify mirror))
     )
-    (fp_circle (center 0 0) (end 25.5 0) (layer "B.SilkS") (width 0.12) (fill none))
     (pad "" np_thru_hole circle (at 31 0) (size 6.4 6.4) (drill 3.2) (layers F&B.Cu *.Mask))
     (pad "" np_thru_hole circle (at -31 0) (size 6.4 6.4) (drill 3.2) (layers F&B.Cu *.Mask))
@@
   (segment (start 52.155689 108.455689) (end 52.75 109.05) (width 0.6096) (layer "In2.Cu") (net 1))
   (segment (start 52.75 109.05) (end 52.75 110.25) (width 0.6096) (layer "In2.Cu") (net 1))
+  (segment (start 58.0605 117.9395) (end 61.5 114.5) (width 0.25) (layer "F.Cu") (net 2))
   (segment (start 92.8 86.375) (end 93.7125 86.375) (width 0.25) (layer "F.Cu") (net 2))
   (segment (start 92.2225 83.525) (end 92.2125 83.515) (width 0.25) (layer "F.Cu") (net 2))
   (segment (start 53.43 78.945) (end 50.955 78.945) (width 0.6096) (layer "F.Cu") (net 2))
+  (segment (start 57.452397 117.9395) (end 58.0605 117.9395) (width 0.25) (layer "F.Cu") (net 2))
   (segment (start 63.5744 110.8056) (end 64.4856 110.8056) (width 0.2) (layer "F.Cu") (net 2))
   (segment (start 91.11 85.02) (end 91.6375 85.5475) (width 0.25) (layer "F.Cu") (net 2))
-  (segment (start 48.6 115.05) (end 48.608 115.042) (width 0.25) (layer "F.Cu") (net 2))
   (segment (start 94.0625 86.875) (end 94.2125 86.725) (width 0.25) (layer "F.Cu") (net 2))
   (segment (start 92.8 86.875) (end 94.0625 86.875) (width 0.25) (layer "F.Cu") (net 2))
   (segment (start 93.7125 86.375) (end 94.2125 85.875) (width 0.25) (layer "F.Cu") (net 2))
   (segment (start 47.5 89.9) (end 47.55 89.85) (width 0.29337) (layer "F.Cu") (net 2))
-  (segment (start 48.608 115.042) (end 51.909999 115.042) (width 0.25) (layer "F.Cu") (net 2))
+  (segment (start 51.909999 116.987) (end 52.862499 117.9395) (width 0.25) (layer "F.Cu") (net 2))
   (segment (start 55.75 127.9) (end 55.749999 127.027) (width 0.25) (layer "F.Cu") (net 2))
   (segment (start 92.8 87.375) (end 94.0625 87.375) (width 0.25) (layer "F.Cu") (net 2))
   (segment (start 94.0625 87.375) (end 94.2125 87.525) (width 0.25) (layer "F.Cu") (net 2))
+  (segment (start 51.909999 115.042) (end 51.909999 116.987) (width 0.25) (layer "F.Cu") (net 2))
   (segment (start 62.2985 108.75) (end 61.401499 108.75) (width 0.25) (layer "F.Cu") (net 2))
+  (segment (start 57.452397 121.1145) (end 57.8855 121.1145) (width 0.25) (layer "F.Cu") (net 2))
   (segment (start 63.08 80.82) (end 64.83 80.82) (width 0.6096) (layer "F.Cu") (net 2))
   (segment (start 91.1375 85.0475) (end 91.1375 86.2125) (width 0.25) (layer "F.Cu") (net 2))
@@
   (segment (start 63.5 103.8) (end 63.5 101.9) (width 0.25) (layer "F.Cu") (net 2))
   (segment (start 63.57 110.81) (end 63.5744 110.8056) (width 0.1) (layer "F.Cu") (net 2))
+  (segment (start 57.452397 119.527) (end 60.979397 116) (width 0.25) (layer "F.Cu") (net 2))
   (segment (start 62.45 79.95) (end 63 80.5) (width 0.6096) (layer "F.Cu") (net 2))
   (segment (start 61.401499 108.75) (end 61.378499 108.727) (width 0.25) (layer "F.Cu") (net 2))
@@
   (segment (start 63.5 101.9) (end 63.55 101.85) (width 0.25) (layer "F.Cu") (net 2))
   (segment (start 89.2125 86.875) (end 90.475 86.875) (width 0.25) (layer "F.Cu") (net 2))
+  (segment (start 57.8855 121.1145) (end 61.5 117.5) (width 0.25) (layer "F.Cu") (net 2))
   (segment (start 62.53 79.82) (end 64.83 79.82) (width 0.6096) (layer "F.Cu") (net 2))
   (segment (start 91.2425 83.645) (end 91.3125 83.575) (width 0.25) (layer "F.Cu") (net 2))
@@
   (segment (start 91.6375 85.5475) (end 91.6375 86.2125) (width 0.25) (layer "F.Cu") (net 2))
   (segment (start 93.1625 83.525) (end 92.2225 83.525) (width 0.25) (layer "F.Cu") (net 2))
+  (segment (start 60.979397 116) (end 61.5 116) (width 0.25) (layer "F.Cu") (net 2))
   (segment (start 90.2625 83.645) (end 91.2425 83.645) (width 0.25) (layer "F.Cu") (net 2))
   (segment (start 63.08 78.82) (end 64.83 78.82) (width 0.6096) (layer "F.Cu") (net 2))
+  (segment (start 52.862499 117.9395) (end 51.4476 117.9395) (width 0.25) (layer "F.Cu") (net 2))
   (segment (start 65.8 87.85) (end 63.55 87.85) (width 0.29337) (layer "F.Cu") (net 2))
   (via (at 58.4 111.65) (size 0.58) (drill 0.4) (layers "F.Cu" "B.Cu") (free) (net 2))
@@
   (via (at 63.57 110.81) (size 0.58) (drill 0.4) (layers "F.Cu" "B.Cu") (net 2))
   (via (at 64.5 82.5) (size 0.58) (drill 0.4) (layers "F.Cu" "B.Cu") (free) (net 2))
+  (via (at 61.5 114.5) (size 0.58) (drill 0.4) (layers "F.Cu" "B.Cu") (free) (net 2))
   (via (at 61.378499 108.727) (size 0.58) (drill 0.4) (layers "F.Cu" "B.Cu") (free) (net 2))
   (via (at 93.1625 83.525) (size 0.58) (drill 0.4) (layers "F.Cu" "B.Cu") (free) (net 2))
@@
   (via (at 55.75 127.9) (size 0.58) (drill 0.4) (layers "F.Cu" "B.Cu") (free) (net 2))
   (via (at 123 123) (size 0.58) (drill 0.4) (layers "F.Cu" "B.Cu") (free) (net 2))
+  (via (at 61.5 116) (size 0.58) (drill 0.4) (layers "F.Cu" "B.Cu") (free) (net 2))
   (via (at 102.225 96.95) (size 0.58) (drill 0.4) (layers "F.Cu" "B.Cu") (free) (net 2))
   (via (at 46.228 118.872) (size 0.58) (drill 0.4) (layers "F.Cu" "B.Cu") (free) (net 2))
+  (via (at 61.5 117.5) (size 0.58) (drill 0.4) (layers "F.Cu" "B.Cu") (free) (net 2))
   (via (at 91.3125 83.575) (size 0.58) (drill 0.4) (layers "F.Cu" "B.Cu") (free) (net 2))
-  (via (at 48.6 115.05) (size 0.58) (drill 0.4) (layers "F.Cu" "B.Cu") (free) (net 2))
   (via (at 50.8 78.92) (size 0.8) (drill 0.4) (layers "F.Cu" "B.Cu") (net 2))
   (via (at 68 86.5) (size 0.58) (drill 0.4) (layers "F.Cu" "B.Cu") (free) (net 2))
@@
     )
   )
-  (zone (net 0) (net_name "") (layers F&B.Cu) (hatch edge 0.508)
+  (zone (net 0) (net_name "") (layers "F.Cu" "In1.Cu" "In2.Cu" "B.Cu") (hatch edge 0.508)
     (connect_pads (clearance 0))
     (min_thickness 0.254)
@@
     )
   )
-  (zone (net 0) (net_name "") (layer "F.Cu") (hatch edge 0.508)
+  (zone (net 0) (net_name "") (layers "F.Cu" "In1.Cu" "In2.Cu" "B.Cu") (hatch edge 0.508)
     (connect_pads (clearance 0))
     (min_thickness 0.254)
